File: KiCad/simple/simple.kicad_sch (KiCad schematic)
At the start: 13 parts, among them IC1 PIC16F15213T-I_SN, J1 Conn_01x02, J2 Conn_01x02, J3 Conn_01x01, J4 Conn_01x02, J5 Conn_01x02, SW1 SW_Push

Commit message: Fix the footprint of C1
Parts:
- C1: footprint Resistor_SMD:R_0603_1608Metric_Pad0.98x0.95mm_HandSolder -> Capacitor_SMD:C_0603_1608Metric
Changed lines of the file:
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@@
       (effects (font (size 1.27 1.27)) (justify left))
     )
-    (property "Footprint" "Resistor_SMD:R_0603_1608Metric_Pad0.98x0.95mm_HandSolder" (at 102.5652 83.82 0)
+    (property "Footprint" "Capacitor_SMD:C_0603_1608Metric" (at 102.5652 83.82 0)
       (effects (font (size 1.27 1.27)) hide)
     )
